File: project files/STM8-Nano.kicad_pcb (KiCad board)
At the start: 2 copper layers, 43.2 x 17.8 mm, 29 parts, among them J1 RIGHT, J2 LEFT, J3 USB_C_Receptacle, J4 SWIM, SW1 RESET, SW2 VCC, U1 STM8F105K4, U2 CH340E, Y1 16MHZ

Commit message: added annotation
Parts:
- removed C7: 1uF, Capacitor_SMD:C_0603_1608Metric
- removed C8: 100nF, Capacitor_SMD:C_0603_1608Metric
- removed REF**: OSHW-Symbol_8.9x8mm_SilkScreen, Symbol:OSHW-Symbol_8.9x8mm_SilkScreen
- added C9: 10uF, Capacitor_SMD:C_0603_1608Metric, F.Cu at (66.0, 100.3)
- D2: value TX -> TX↓
- J3: value USB_C_Receptacle -> USB_C_Receptacle_USB2.0
- turned C2 to 180 degrees
Connections:
- J4 pad 3: /~{RST} -> GND
- J4 pad 4: GND -> /~{RST}
- U1 pad 7: VDDA -> VCC
- U2 pad 4: unconnected-(U2-Pad4) -> Net-(C9-Pad1)
- U2 pad 7: VCC -> +5V
Other:
- board text added: "RX0 ↓"
- board text added: "TX0 ↑"
- board text removed: "↑ TX0"
- board text removed: "↓ RX0"

Commit message: case change
Parts:
- removed R7: 0R, Resistor_SMD:R_0805_2012Metric
- C1, C3, C4, C5, C6, C9: footprint Capacitor_SMD:C_0603_1608Metric -> Capacitor_SMD:C_0402_1005Metric
- D1, D2, D3, D4: footprint LED_SMD:LED_0603_1608Metric -> LED_SMD:LED_0402_1005Metric
- R1, R2, R3, R4, R5, R6: footprint Resistor_SMD:R_0603_1608Metric_Pad0.98x0.95mm_HandSolder -> Resistor_SMD:R_0402_1005Metric
- moved SW1 19.7 mm to (66.7, 89.5)
- moved C9 13.3 mm to (61.2, 87.9), turned to -90 degrees
- moved C1 2.62 mm to (80.0, 89.5)
- moved D2 2.01 mm to (85.1, 83.2)
- moved R4 1.91 mm to (82.5, 83.2)
- moved R1 1.82 mm to (59.2, 87.9), turned to -90 degrees
- moved R2 1.82 mm to (59.2, 82.3), turned to 90 degrees
- moved D1 1.42 mm to (85.1, 84.5)
- moved R3 1.27 mm to (82.5, 84.5)
- moved D4 0.90 mm to (85.1, 85.7)
- moved D3 0.63 mm to (85.1, 87.0)
- moved R6 0.63 mm to (82.5, 85.7)
- moved Y1 0.30 mm to (67.3, 83.5)
Routing:
- net USB(+): track 2.78 -> 0.00 mm
- net USB(-): track 2.78 -> 0.00 mm

Commit message: up
Parts:
- SW2: footprint Jumper:SolderJumper-3_P2.0mm_Open_TrianglePad1.0x1.5mm_NumberLabels -> Button_Switch_SMD:SW_SPDT_PCM12
- moved SW2 15.1 mm to (91.8, 85.1), turned to 90 degrees
- moved J4 6.35 mm to (86.4, 81.3)
Connections:
- net Net-(J3-PadA4) renamed VBUS

Commit message: LED moved
Other:
- board text added: "RX↓"
- board text added: "TX↑"
- board text removed: "RX0 ↓"
- board text removed: "TX0 ↑"
Changed lines of the file:
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@@
     (effects (font (size 0.75 0.75) (thickness 0.15)))
   )
-  (gr_text "RX0\n↓" (at 87.63 80.01) (layer "F.SilkS")
+  (gr_text "RX↓" (at 87.63 79.375) (layer "F.SilkS")
     (effects (font (size 0.75 0.75) (thickness 0.15)))
   )
@@
     (effects (font (size 0.75 0.75) (thickness 0.15)))
   )
-  (gr_text "TX0\n↑" (at 90.17 80.01) (layer "F.SilkS")
+  (gr_text "TX↑" (at 90.17 79.375) (layer "F.SilkS")
     (effects (font (size 0.75 0.75) (thickness 0.15)))
   )
@@
     (pts (xy 52.07 77.47) (xy 52.07 92.71))
     (height 20.32)
-    (gr_text "0,6000 in" (at 30.6 85.09 90) (layer "Dwgs.User")
+    (gr_text "15,2400 mm" (at 30.6 85.09 90) (layer "Dwgs.User")
       (effects (font (size 1 1) (thickness 0.15)))
     )
@@
     (pts (xy 50.8 93.98) (xy 93.98 93.98))
     (height 20.32)
-    (gr_text "1,7000 in" (at 72.39 113.15) (layer "Dwgs.User")
+    (gr_text "43,1800 mm" (at 72.39 113.15) (layer "Dwgs.User")
       (effects (font (size 1 1) (thickness 0.15)))
     )
@@
     (pts (xy 93.98 76.2) (xy 93.98 93.98))
     (height -20.32)
-    (gr_text "0,7000 in" (at 113.15 85.09 90) (layer "Dwgs.User")
+    (gr_text "17,7800 mm" (at 113.15 85.09 90) (layer "Dwgs.User")
       (effects (font (size 1 1) (thickness 0.15)))
     )
@@
     (pts (xy 52.07 77.47) (xy 92.71 77.47))
     (height -13.97)
-    (gr_text "1,6000 in" (at 72.39 62.35) (layer "Dwgs.User")
+    (gr_text "40,6400 mm" (at 72.39 62.35) (layer "Dwgs.User")
       (effects (font (size 1 1) (thickness 0.15)))
     )
